Commit message: adding mesh files

File: section02_skeleton/ros_gazebo_skeleton/ros_urdf/urdf/step_05.urdf (robot description, URDF)
Before this commit: robot visual, 16 links, 15 joints
Links:
- link left_gripper: geometry visual mesh filename=package://ros_urdf/meshes/l_finger.dae
- link left_tip: geometry visual mesh filename=package://ros_urdf/meshes/l_finger_tip.dae
- link right_gripper: geometry visual mesh filename=package://ros_urdf/meshes/l_finger.dae
- link right_tip: geometry visual mesh filename=package://ros_urdf/meshes/l_finger_tip.dae

File: section02_skeleton/ros_gazebo_skeleton/ros_urdf/urdf/step_06.urdf (robot description, URDF)
Before this commit: robot visual, 16 links, 15 joints
Links:
- link left_gripper: geometry visual mesh filename=package://ros_urdf/meshes/l_finger.dae
- link left_tip: geometry visual mesh filename=package://ros_urdf/meshes/l_finger_tip.dae
- link right_gripper: geometry visual mesh filename=package://ros_urdf/meshes/l_finger.dae
- link right_tip: geometry visual mesh filename=package://ros_urdf/meshes/l_finger_tip.dae
