Commit message: adding urdf changes

File: section02_skeleton/ros_gazebo_skeleton/ros_urdf/urdf/step_01.urdf (robot description, URDF)
Before this commit: robot myfirst, 1 links, 0 joints
Links:
- added link right_bar; visual box size=0.2 0.4 0.5
Joints:
- added joint my_joint: type fixed, parent base_link, child right_bar, origin xyz=0 0 1 rpy=0 0 3.1416

File: section02_skeleton/ros_gazebo_skeleton/ros_urdf/urdf/step_03.urdf (robot description, URDF)
Before this commit: robot origins, 2 links, 1 joints
Links:
- added link left_leg; visual box size=0.6 0.1 0.2
Joints:
- added joint base_to_left_leg: type fixed, parent base_link, child left_leg, origin xyz=0 -0.22 0.25
